Commit message: feat(roverrobotics_description): add RGBD camera

File: roverrobotics_description/urdf/accessories/rgbd_camera.urdf (robot description, URDF)
Before this commit: robot None, 2 links, 2 joints
Links:
- removed link depth_camera_link
- removed link depth_camera_link_optical
- added link rgbd_camera_link; visual box size=0.01 0.03 0.03
- added link rgbd_camera_link_optical
Joints:
- removed joint depth_camera_to_payload
- added joint rgbd_camera_to_payload: type fixed, parent payload_link, child rgbd_camera_link, origin xyz=0.174 0 0.15 rpy=0 0 0
- joint depth_camera_optical_joint: child depth_camera_link_optical -> rgbd_camera_link_optical; parent depth_camera_link -> rgbd_camera_link
