Commit message: style(roverrobotics_description): make RGB-D camera link transparent

File: roverrobotics_description/urdf/accessories/rgbd_camera.urdf (robot description, URDF)
Before this commit: robot rgbd_camera, 2 links, 2 joints
Links:
- link rgbd_camera_link: geometry visual box size=0.005 0.03 0.03
