Commit message: feat(actor_command_plugin, roverrobotics_description/meshes): add plugin to control actor via cmd_vel or path and publish distances and positions. Update meshes.
Includes:
- New actor_command_plugin with support for cmd_vel-based or path-based control (WIP for path mode)
- Publishing of actor position, model or link pose, and distance between them
- Meshes and URDF updates and new accessories links

File: roverrobotics_description/urdf/accessories/depth_camera.urdf (robot description, URDF)
Before this commit: robot None, 2 links, 2 joints
Joints:
- removed joint depth_camera_to_payload
- added joint depth_camera_to_soporte_camaras: type fixed, parent soporte_camaras, child depth_camera_link, origin xyz=0.174 0 0.15 rpy=0 0 0

File: roverrobotics_description/urdf/accessories/rgbd_camera.urdf (robot description, URDF)
Before this commit: robot None, 2 links, 2 joints
Links:
- link rgbd_camera_link: geometry visual box size=0.005 0.03 0.03
Joints:
- removed joint rgbd_camera_to_payload
- added joint rgbd_camera_to_soporte_camaras: type fixed, parent soporte_camaras, child rgbd_camera_link, origin xyz=0.054356 0 0.055118 rpy=0 ${-3.14159/18} 0

File: roverrobotics_description/urdf/accessories/rover_dev_payload.urdf (robot description, URDF)
Before this commit: robot rover_miti_payload, 1 links, 1 joints
Links:
- link payload_link: geometry collision mesh filename=file://$(find roverrobotics_description)/meshes/Payload_col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; visual mesh filename=file://$(find roverrobotics_description)/meshes/Payload_col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

File: roverrobotics_description/urdf/accessories/rplidar_s2.urdf (robot description, URDF)
Before this commit: robot rplidar_s2, 1 links, 1 joints
Joints:
- joint lidar_to_payload: origin xyz=0.174 0 0.10 rpy=0 0 3.1415 -> xyz=0 0 0.10 rpy=0 0 3.1415

File: roverrobotics_description/urdf/mini.urdf (robot description, URDF)
Before this commit: robot rover_mini, 6 links, 5 joints
Links:
- link fl_wheel_link: geometry collision mesh filename=file://$(find roverrobotics_description)/meshes/65wheels_co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; visual mesh filename=file://$(find roverrobotics_description)/meshes/65wheels_co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
- link fr_wheel_link: geometry collision mesh filename=file://$(find roverrobotics_description)/meshes/65wheels_co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; visual mesh filename=file://$(find roverrobotics_description)/meshes/65wheels_co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
- link rl_wheel_link: geometry collision mesh filename=file://$(find roverrobotics_description)/meshes/65wheels_co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; visual mesh filename=file://$(find roverrobotics_description)/meshes/65wheels_co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
- link rr_wheel_link: geometry collision mesh filename=file://$(find roverrobotics_description)/meshes/65wheels_co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; visual mesh filename=file://$(find roverrobotics_description)/meshes/65wheels_co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
