Commit message: feat(roverrobotics_description): add stereo_camera sensors for oak_d_lite, and change to revolute joint soporte_camaras_to_base_columnas for dinamixel simulation

File: roverrobotics_description/urdf/accessories/base_columnas.urdf (robot description, URDF)
Before this commit: robot rover_mini_base_columnas, 1 links, 1 joints
Links:
- link base_columnas: geometry collision mesh filename=file://$(find roverrobotics_description)/meshes/ColumnasBas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; visual mesh filename=file://$(find roverrobotics_description)/meshes/ColumnasBas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

File: roverrobotics_description/urdf/accessories/soporte_camaras.urdf (robot description, URDF)
Before this commit: robot rover_mini_soporte_camaras, 1 links, 1 joints
Links:
- link soporte_camaras: mass None -> 2.95; geometry collision mesh filename=file://$(find roverrobotics_description)/meshes/Soportes_ca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; visual mesh filename=file://$(find roverrobotics_description)/meshes/Soportes_ca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
Joints:
- joint soporte_camaras_to_base_columnas: axis (none) -> 0 0 1; limit (none) -> lower=-1.5708 upper=1.5708 effort=5.0 velocity=2.0; type fixed -> revolute

Commit message: feat(roverrobotics_description): update robot meshes, joints, camera intrinsics
Includes:
- Updated base_columnas visual mesh removing attached lidar and adding dynamixel model (ColumnasConDyna0_001.dae)
- Fixed base_columnas collision orientation
- Updated rplidar_s2 visual mesh to avoid flipped lidar orientation (Lidar_sin_girar.dae)
- Changed soporte_camaras joint type from fixed to revolute
- Added pure delay configuration tags to mini.urdf dynamics plugin
- Added base_footprint link for SLAM/Nav2 compatibility to mini.urdf
- Added RGB-D camera intrinsics parameters

File: roverrobotics_description/urdf/accessories/base_columnas.urdf (robot description, URDF)
Before this commit: robot rover_mini_base_columnas, 1 links, 1 joints
Links:
- link base_columnas: geometry collision mesh filename=file://$(find roverrobotics_description)/meshes/ColumnasCon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; visual mesh filename=file://$(find roverrobotics_description)/meshes/ColumnasCon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

File: roverrobotics_description/urdf/accessories/rgbd_camera.urdf (robot description, URDF)
Before this commit: robot None, 2 links, 2 joints
Joints:
- joint rgbd_camera_to_soporte_camaras: origin xyz=0.054356 0 0.055118 rpy=0 ${-3.14159/18} 0 -> xyz=-0.054356 0 0.055118 rpy=0 ${-3.14159/18} 3.14159

File: roverrobotics_description/urdf/accessories/rplidar_s2.urdf (robot description, URDF)
Before this commit: robot rplidar_s2, 1 links, 1 joints
Links:
- link lidar_link: geometry collision mesh filename=file://$(find roverrobotics_description)/meshes/Lidar_sin_g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; visual mesh filename=file://$(find roverrobotics_description)/meshes/Lidar_sin_g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

File: roverrobotics_description/urdf/accessories/soporte_camaras.urdf (robot description, URDF)
Before this commit: robot rover_mini_soporte_camaras, 1 links, 1 joints
Links:
- link soporte_camaras: mass None -> 2.95; geometry collision mesh filename=file://$(find roverrobotics_description)/meshes/Soportes_ca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; visual mesh filename=file://$(find roverrobotics_description)/meshes/Soportes_ca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
Joints:
- joint soporte_camaras_to_base_columnas: axis (none) -> 0 0 1; limit (none) -> lower=-1.5708 upper=1.5708 effort=5.0 velocity=2.0; type fixed -> revolute

File: roverrobotics_description/urdf/mini.urdf (robot description, URDF)
Before this commit: robot rover_mini, 6 links, 5 joints
Links:
- added link base_footprint
Joints:
- added joint base_footprint_joint: type fixed, parent base_link, child base_footprint, origin xyz=0 0 0 rpy=0 0 0

Commit message: feat(roverrobotics_description): add wheel visual details and split Oak and Orbbec models

File: roverrobotics_description/urdf/accessories/base_columnas.urdf (robot description, URDF)
Before this commit: robot rover_mini_base_columnas, 1 links, 1 joints
Links:
- link base_columnas: geometry collision mesh filename=file://$(find roverrobotics_description)/meshes/ColumnasBas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; visual mesh filename=file://$(find roverrobotics_description)/meshes/ColumnasBas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

File: roverrobotics_description/urdf/accessories/rgbd_camera.urdf (robot description, URDF)
Before this commit: robot None, 2 links, 2 joints
Joints:
- removed joint rgbd_camera_to_soporte_camaras
- added joint rgbd_camera_to_soporte_camaras_orbec: type fixed, parent soporte_camaras_orbec, child rgbd_camera_link, origin xyz=-0.054356 0 0.055118 rpy=0 ${-3.14159/18} 3.14159

File: roverrobotics_description/urdf/accessories/soporte_camaras.urdf (robot description, URDF)
Before this commit: robot rover_mini_soporte_camaras, 1 links, 1 joints
Links:
- removed link soporte_camaras
- added link soporte_camaras_orbec, mass 2.95; collision mesh filename=file://$(find roverrobotics_description)/meshes/Soporte_con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; visual mesh filename=file://$(find roverrobotics_description)/meshes/Soporte_con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
Joints:
- joint soporte_camaras_to_base_columnas: child soporte_camaras -> soporte_camaras_orbec

File: roverrobotics_description/urdf/mini.urdf (robot description, URDF)
Before this commit: robot rover_mini, 7 links, 6 joints
Links:
- link fl_wheel_link: geometry collision mesh filename=file://$(find roverrobotics_description)/meshes/wheel.dae; visual mesh filename=file://$(find roverrobotics_description)/meshes/wheel.dae
- link fr_wheel_link: geometry collision mesh filename=file://$(find roverrobotics_description)/meshes/wheel.dae; visual mesh filename=file://$(find roverrobotics_description)/meshes/wheel.dae
- link rl_wheel_link: geometry collision mesh filename=file://$(find roverrobotics_description)/meshes/wheel.dae; visual mesh filename=file://$(find roverrobotics_description)/meshes/wheel.dae
- link rr_wheel_link: geometry collision mesh filename=file://$(find roverrobotics_description)/meshes/wheel.dae; visual mesh filename=file://$(find roverrobotics_description)/meshes/wheel.dae

Commit message: fix(roverrobotics_description): relocate base_columnas Z offsets from visuals to joints

File: roverrobotics_description/urdf/accessories/base_columnas.urdf (robot description, URDF)
Before this commit: robot rover_mini_base_columnas, 1 links, 1 joints
Joints:
- joint base_columnas_to_payload: origin xyz=0 0 0 -> xyz=0 0 0.194

File: roverrobotics_description/urdf/accessories/dynamixel.urdf (robot description, URDF)
Before this commit: robot rover_mini_dynamixel, 1 links, 1 joints
Joints:
- joint dynamixel_to_base_columnas: origin xyz=0 0 0 -> xyz=0 0 -0.011

File: roverrobotics_description/urdf/accessories/soporte_camaras.urdf (robot description, URDF)
Before this commit: robot rover_mini_soporte_camaras_orbec, 1 links, 1 joints
Joints:
- joint soporte_camaras_to_base_columnas: origin xyz=0 0 0.182 -> xyz=0 0 -0.012

Commit message: fix(roverrobotics_description): update orientations after base_columnas rotation change

File: roverrobotics_description/urdf/accessories/base_columnas.urdf (robot description, URDF)
Before this commit: robot rover_mini_base_columnas, 1 links, 1 joints
Joints:
- joint base_columnas_to_payload: origin xyz=0 0 0.194 -> xyz=0 0 0.19376 rpy=0 0 3.14159

File: roverrobotics_description/urdf/accessories/dynamixel.urdf (robot description, URDF)
Before this commit: robot rover_mini_dynamixel, 1 links, 1 joints
Joints:
- joint dynamixel_to_base_columnas: origin xyz=0 0 -0.011 -> xyz=0 0 -0.0111

File: roverrobotics_description/urdf/accessories/rgbd_camera.urdf (robot description, URDF)
Before this commit: robot None, 2 links, 2 joints
Joints:
- joint rgbd_camera_to_soporte_camaras_orbec: origin xyz=-0.054356 0 0.055118 rpy=0 ${-3.14159/18} 3.14159 -> xyz=0.054356 0 0.055118 rpy=0 ${-3.14159/18} 0

File: roverrobotics_description/urdf/accessories/soporte_camaras.urdf (robot description, URDF)
Before this commit: robot rover_mini_soporte_camaras_orbec, 1 links, 1 joints
Joints:
- joint soporte_camaras_to_base_columnas: origin xyz=0 0 -0.012 -> xyz=0 0 -0.01196 rpy=0 0 0
