Commit message: refactor(roverrobotics_description): move camera rotation joint to dynamixel
- Add new link for the rotating part of the dynamixel motor
- Move the controlled joint from soporte_camaras to dynamixel.urdf
- New dynamixel_top_to_dynamixel revolute joint as the new rotation axis
- Rename soporte_camaras_to_base_columnas to soporte_camaras_to_dynamixel_top
- Convert the camera support attachment joint from revolute to fixed

File: roverrobotics_description/urdf/accessories/dynamixel.urdf (robot description, URDF)
Before this commit: robot rover_mini_dynamixel, 1 links, 1 joints
Links:
- added link dynamixel_top; visual mesh filename=file://$(find roverrobotics_description)/meshes/Dynamixel_t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
Joints:
- added joint dynamixel_top_to_dynamixel: type revolute, parent dynamixel, child dynamixel_top, origin xyz=0 0 0, axis 0 0 1, limit lower=-1.5708 upper=1.5708 effort=5.0 velocity=2.0

File: roverrobotics_description/urdf/accessories/soporte_camaras.urdf (robot description, URDF)
Before this commit: robot rover_mini_soporte_camaras_orbec, 1 links, 1 joints
Joints:
- removed joint soporte_camaras_to_base_columnas
- added joint soporte_camaras_to_dynamixel_top: type fixed, parent dynamixel_top, child soporte_camaras_orbec, origin xyz=0 0 -0.00086 rpy=0 0 0
