Commit message: refactor(roverrobotics_description): standardize URDF, link, joint and mesh naming
- Rename robot description files and meshes using consistent English names
- Rename links and joints to follow a consistent naming convention
- Update mesh references, xacro includes and dependent joint references
- Remove obsolete and superseded mesh files
- Improve naming consistency across the existing robot description

File: roverrobotics_description/urdf/accessories/dynamixel.urdf (robot description, URDF)
Before this commit: robot dynamixel, 2 links, 2 joints
Links:
- removed link dynamixel
- removed link dynamixel_top
- added link dynamixel_link; collision mesh filename=file://$(find roverrobotics_description)/meshes/Dynamixel.d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; visual mesh filename=file://$(find roverrobotics_description)/meshes/Dynamixel.d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
- added link dynamixel_top_link; collision mesh filename=file://$(find roverrobotics_description)/meshes/Dynamixel_t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; visual mesh filename=file://$(find roverrobotics_description)/meshes/Dynamixel_t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
Joints:
- removed joint dynamixel_to_base_columnas
- added joint dynamixel_to_camera_riser: type fixed, parent camera_riser_link, child dynamixel_link, origin xyz=0 0 -0.0111
- joint dynamixel_top_to_dynamixel: child dynamixel_top -> dynamixel_top_link; parent dynamixel -> dynamixel_link

File: roverrobotics_description/urdf/accessories/oak.urdf (robot description, URDF)
Before this commit: robot oak, 1 links, 1 joints
Links:
- removed link oak
- added link oak_link; collision mesh filename=file://$(find roverrobotics_description)/meshes/Oak.dae; visual mesh filename=file://$(find roverrobotics_description)/meshes/Oak.dae
Joints:
- removed joint oak_to_soporte_camaras_orbbec
- added joint oak_to_orbbec_camera_assembly: type fixed, parent orbbec_camera_assembly_link, child oak_link, origin xyz=-0.03296 0 0.06407 rpy=0 0 0

File: roverrobotics_description/urdf/accessories/rgbd_camera.urdf (robot description, URDF)
Before this commit: robot rgbd_camera, 2 links, 2 joints
Links:
- removed link rgbd_camera_link_optical
- added link rgbd_camera_optical_link
- link rgbd_camera_link: geometry 
Joints:
- removed joint depth_camera_optical_joint
- removed joint rgbd_camera_to_soporte_camaras_orbbec
- added joint rgbd_camera_optical_joint: type fixed, parent rgbd_camera_link, child rgbd_camera_optical_link, origin xyz=0 0 0 rpy=${-3.14159/2} 0 ${-3.14159/2}
- added joint rgbd_camera_to_orbbec_camera_assembly: type fixed, parent orbbec_camera_assembly_link, child rgbd_camera_link, origin xyz=0 0 0 rpy=0 ${-3.14159/18} 0

File: roverrobotics_description/urdf/accessories/rover_dev_payload.urdf (robot description, URDF)
Before this commit: robot rover_dev_payload, 1 links, 1 joints
Links:
- link payload_link: geometry collision mesh filename=file://$(find roverrobotics_description)/meshes/Payload.dae; visual mesh filename=file://$(find roverrobotics_description)/meshes/Payload.dae

File: roverrobotics_description/urdf/accessories/rplidar_s2.urdf (robot description, URDF)
Before this commit: robot rplidar_s2, 1 links, 1 joints
Links:
- link lidar_link: geometry collision mesh filename=file://$(find roverrobotics_description)/meshes/LiDAR.dae; visual mesh filename=file://$(find roverrobotics_description)/meshes/LiDAR.dae

File: roverrobotics_description/urdf/mini.urdf (robot description, URDF)
Before this commit: robot rover_mini, 6 links, 5 joints
Links:
- link chassis_link: geometry collision mesh filename=file://$(find roverrobotics_description)/meshes/MiniChassis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; visual mesh filename=file://$(find roverrobotics_description)/meshes/MiniChassis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
- link fl_wheel_link: geometry collision mesh filename=file://$(find roverrobotics_description)/meshes/Wheel.dae; visual mesh filename=file://$(find roverrobotics_description)/meshes/Wheel.dae
- link fr_wheel_link: geometry collision mesh filename=file://$(find roverrobotics_description)/meshes/Wheel.dae; visual mesh filename=file://$(find roverrobotics_description)/meshes/Wheel.dae
- link rl_wheel_link: geometry collision mesh filename=file://$(find roverrobotics_description)/meshes/Wheel.dae; visual mesh filename=file://$(find roverrobotics_description)/meshes/Wheel.dae
- link rr_wheel_link: geometry collision mesh filename=file://$(find roverrobotics_description)/meshes/Wheel.dae; visual mesh filename=file://$(find roverrobotics_description)/meshes/Wheel.dae
