Commit message: refactor(roverrobotics_description):relocate Orbbec and OAK camera joints to their corresponding sensor axes

File: roverrobotics_description/urdf/accessories/oak.urdf (robot description, URDF)
Before this commit: robot rover_mini_oak, 1 links, 1 joints
Joints:
- joint oak_to_soporte_camaras_orbec: origin xyz=0 0 0 -> xyz=-0.03296 0 0.06407 rpy=0 0 0

File: roverrobotics_description/urdf/accessories/rgbd_camera.urdf (robot description, URDF)
Before this commit: robot None, 2 links, 2 joints
Joints:
- joint rgbd_camera_to_soporte_camaras_orbec: origin xyz=0.054356 0 0.055118 rpy=0 ${-3.14159/18} 0 -> xyz=0 0 0 rpy=0 ${-3.14159/18} 0

File: roverrobotics_description/urdf/accessories/rplidar_s2.urdf (robot description, URDF)
Before this commit: robot rplidar_s2, 1 links, 1 joints
Joints:
- joint lidar_to_payload: origin xyz=0 0 0.10 rpy=0 0 3.1415 -> xyz=0 0 0.10315 rpy=0 0 3.1415

File: roverrobotics_description/urdf/accessories/soporte_camaras.urdf (robot description, URDF)
Before this commit: robot rover_mini_soporte_camaras_orbec, 1 links, 1 joints
Joints:
- joint soporte_camaras_to_dynamixel_top: origin xyz=0 0 -0.00086 rpy=0 0 0 -> xyz=0.05509 0 0.05362 rpy=0 0 0

Commit message: refactor(roverrobotics_description): remove base_footprint and clean up sensor definitions
- Remove the base_footprint link from the robot description
- Rename Orbec references to Orbbec
- Update related URDF definitions after the naming change
- Adjust collision poses where required
- Improve consistency of the robot model

File: roverrobotics_description/urdf/accessories/oak.urdf (robot description, URDF)
Before this commit: robot rover_mini_oak, 1 links, 1 joints
Joints:
- removed joint oak_to_soporte_camaras_orbec
- added joint oak_to_soporte_camaras_orbbec: type fixed, parent soporte_camaras_orbbec, child oak, origin xyz=-0.03296 0 0.06407 rpy=0 0 0

File: roverrobotics_description/urdf/accessories/rgbd_camera.urdf (robot description, URDF)
Before this commit: robot None, 2 links, 2 joints
Joints:
- removed joint rgbd_camera_to_soporte_camaras_orbec
- added joint rgbd_camera_to_soporte_camaras_orbbec: type fixed, parent soporte_camaras_orbbec, child rgbd_camera_link, origin xyz=0 0 0 rpy=0 ${-3.14159/18} 0

File: roverrobotics_description/urdf/accessories/soporte_camaras.urdf (robot description, URDF)
Before this commit: robot rover_mini_soporte_camaras_orbec, 1 links, 1 joints
Links:
- removed link soporte_camaras_orbec
- added link soporte_camaras_orbbec, mass 2.95; collision mesh filename=file://$(find roverrobotics_description)/meshes/Soporte_con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; visual mesh filename=file://$(find roverrobotics_description)/meshes/Soporte_con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
Joints:
- removed joint soporte_camaras_to_dynamixel_top
- added joint soporte_camaras_orbbec_to_dynamixel_top: type fixed, parent dynamixel_top, child soporte_camaras_orbbec, origin xyz=0.05509 0 0.05362 rpy=0 0 0

File: roverrobotics_description/urdf/mini.urdf (robot description, URDF)
Before this commit: robot rover_mini, 7 links, 6 joints
Links:
- removed link base_footprint
Joints:
- removed joint base_footprint_joint
